File: kicad/init_dawn.d.kicad_pcb (KiCad board)
At the start: 2 copper layers, 113.5 x 80 mm, 14 parts, among them SW4 SW_Push, SW6 SW_Push, SW7 SW_Push, U2 XIAO-ESP32-C3-SMD

Commit message: firmware + minor fixes on pcb
Parts:
- removed H3, H4: MountingHole, MountingHole:MountingHole_3.2mm_M3
- removed SW1, SW2: ~, Button_Switch_Keyboard:SW_Cherry_MX_1.00u_PCB
- moved H1 147.2 mm to (1345.5, 1057.5)
- moved tft_header1 118.0 mm to (1273.5, 1059.8)
- moved U2 105.4 mm to (1300.7, 1073.7)
- moved SW4 103.4 mm to (1333.5, 1079.9)
- moved SW5 102.3 mm to (1312.8, 1079.9)
- moved SW3 101.4 mm to (1333.5, 1058.4)
- moved BZ1 96.3 mm to (1344.2, 1073.0)
- moved SW6 80.1 mm to (1291.5, 1079.9)
- moved H2 77.5 mm to (1274.0, 1088.5)
- moved SW7 64.5 mm to (1292.0, 1057.9)
Connections:
- SW6 pad 2: Net-(BZ1--) -> Net-(U2-D4)
- U2 pad 13: unconnected-(U2-GND-Pad13) -> Net-(BZ1--)
- U2 pad 18: Net-(U2-D2) -> unconnected-(U2-GND-Pad18)
- U2 pad 5: Net-(BZ1--) -> Net-(U2-D4)
Routing:
- net Net-(U2-D3): track 241.8 -> 96.2 mm, vias 1 -> 0
- net Net-(U2-D1): track 133.0 -> 36.2 mm
- net Net-(BZ1-+): track 36.5 -> 129.7 mm
- net Net-(U2-3V3_OUT): track 216.1 -> 146.3 mm, vias 1 -> 0
- net Net-(BZ1--): track 148.6 -> 89.0 mm, vias 0 -> 2
- net Net-(U2-D10): track 14.5 -> 68.7 mm
- net Net-(U2-D7): track 14.3 -> 66.8 mm, vias 0 -> 1
- net Net-(U2-D9/BOOT): track 13.2 -> 53.6 mm, vias 0 -> 1
- net Net-(U2-D5): track 54.0 -> 24.4 mm, vias 1 -> 0
- net Net-(U2-D4): track 0.00 -> 25.1 mm, vias 0 -> 2
- net Net-(U2-D8): track 42.7 -> 61.1 mm
- net Net-(U2-D2): track 79.5 -> 63.5 mm
- net Net-(U2-D0): track 38.5 -> 42.8 mm, vias 0 -> 1
- net (no net): track 0.60 -> 0.00 mm, vias 1 -> 0
Other:
- board size 113.5 x 80 mm -> 83.5 x 45 mm
- board text added: "by Erox-02"
- board text removed: "I use arch btw. - Erox-02"
