File: kicad/init_dawn.d.kicad_sch (KiCad schematic)
At the start: 14 parts, among them SW4 SW_Push, SW6 SW_Push, SW7 SW_Push, U2 XIAO-ESP32-C3-SMD

Commit message: firmware + minor fixes on pcb
Parts:
- removed H3, H4: MountingHole, MountingHole:MountingHole_3.2mm_M3, symbol Mechanical:MountingHole
- removed SW1, SW2: (no value), Button_Switch_Keyboard:SW_Cherry_MX_1.00u_PCB, symbol Switch:SW_Push
Connections:
- net at U2.13 (GND): now also BZ1.2 (-), tft_header1.1 (Pin_1)
- net at SW4.2, U2.3 (D2): no longer U2.18 (GND)
- net at SW6.2, U2.5 (D4): no longer BZ1.2 (-), tft_header1.1 (Pin_1)
